File: KiCAD/Sender_Receiver.kicad_sch (KiCad schematic)
At the start: 43 parts, among them J1 1-wire, J11 3, J12 12, J13 IOB, J14 IOA, J15 IO, J16 GND, J17 Signal (yellow), J18 Gnd (black), J2 1-wire, Q2 FQP27P06, SW2 Debug Mode, U2 I2C-to-1-Wire bridge, U3 Solar Charger, U6 LM339

Commit message: modified documents and Kicad drawing
Parts:
- added JP4: Activate OLED for 30 sec., symbol Jumper:Jumper_2_Open
- SW3, U1, U7, Water_Contact_Lower1, Water_Contact_Upper1: value ~ -> (none)
Connections:
- net GND: now also JP4.2 (B)
- net at U3. (Sys_Out_+): now also C1.2, U1. (Batt_-); no longer SP. (-)
- new net: R2.2, U1.7 (RST), U2. (Vin)
- new net: SP. (-), U3. (Sys_Out_+)
- new net: JP4.1 (A), U7.18 (GPIO19)
- new net: R1.2, U1.8 (GPIO00), U2. (Vin)
- new net: C1.1, U1. (Batt_-), U3. (Sys_Out_+)
- now unconnected: U1.7 (RST), U1.8 (GPIO00)
- no-connect marks 59 -> 58
